File: Projekti_iz_elektronike/Vsebine/Študijsko_Gradivo/circ/1_1_Darlingtom_open_collector.kicad_sch (KiCad schematic)
At the start: 8 parts, among them Q1 NPN, Q2 NPN

Commit message: ročno razžagovanje
Parts:
- added R3: 7.2k, symbol Device:R
- added R4: 2.7k, symbol Device:R
Connections:
- net GND: now also R4.2
- net at Q1.2 (B), Q2.3 (E): now also R3.2, R4.1
- net at Q2.2 (B), R2.2: now also R3.1
Changed lines of the file:
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@@
   (junction (at 54.61 46.99) (diameter 0) (color 0 0 0 0)
   )
+  (junction (at 74.93 46.99) (diameter 0) (color 0 0 0 0)
+  )
+  (junction (at 83.82 62.23) (diameter 0) (color 0 0 0 0)
+  )
+  (junction (at 97.79 62.23) (diameter 0) (color 0 0 0 0)
+  )
+  (junction (at 83.82 52.07) (diameter 0) (color 0 0 0 0)
+  )
   (wire (pts (xy 38.1 81.28) (xy 38.1 83.82))
     (stroke (width 0) (type default))
@@
     (stroke (width 0) (type default))
   )
+  (wire (pts (xy 74.93 46.99) (xy 74.93 62.23))
+    (stroke (width 0) (type default))
+  )
   (wire (pts (xy 54.61 72.39) (xy 97.79 72.39))
     (stroke (width 0) (type default))
@@
     (stroke (width 0) (type default))
   )
+  (wire (pts (xy 97.79 62.23) (xy 97.79 72.39))
+    (stroke (width 0) (type default))
+  )
+  (wire (pts (xy 74.93 46.99) (xy 76.2 46.99))
+    (stroke (width 0) (type default))
+  )
   (wire (pts (xy 133.35 27.94) (xy 133.35 30.48))
     (stroke (width 0) (type default))
@@
     (stroke (width 0) (type default))
   )
-  (wire (pts (xy 71.12 46.99) (xy 76.2 46.99))
+  (wire (pts (xy 83.82 62.23) (xy 86.36 62.23))
+    (stroke (width 0) (type default))
+  )
+  (wire (pts (xy 71.12 46.99) (xy 74.93 46.99))
     (stroke (width 0) (type default))
   )
@@
     (stroke (width 0) (type default))
   )
+  (wire (pts (xy 83.82 52.07) (xy 83.82 62.23))
+    (stroke (width 0) (type default))
+  )
+  (wire (pts (xy 93.98 62.23) (xy 97.79 62.23))
+    (stroke (width 0) (type default))
+  )
   (wire (pts (xy 54.61 58.42) (xy 54.61 72.39))
     (stroke (width 0) (type default))
@@
     (stroke (width 0) (type default))
   )
-  (wire (pts (xy 97.79 57.15) (xy 97.79 72.39))
+  (wire (pts (xy 97.79 57.15) (xy 97.79 62.23))
+    (stroke (width 0) (type default))
+  )
+  (wire (pts (xy 82.55 62.23) (xy 83.82 62.23))
     (stroke (width 0) (type default))
   )
@@
         )
       )
+    )
+  )
+  (symbol (lib_id "Device:R") (at 90.17 62.23 90) (unit 1)
+    (in_bom yes) (on_board yes) (dnp no) (fields_autoplaced)
+    (property "Reference" "R4" (at 90.17 55.88 90)
+      (effects (font (size 1.27 1.27)))
+    )
+    (property "Value" "2.7k" (at 90.17 58.42 90)
+      (effects (font (size 1.27 1.27)))
+    )
+    (property "Footprint" "" (at 90.17 64.008 90)
+      (effects (font (size 1.27 1.27)) hide)
+    )
+    (property "Datasheet" "~" (at 90.17 62.23 0)
+      (effects (font (size 1.27 1.27)) hide)
+    )
+    (pin "1")
+    (pin "2")
+    (instances
+      (project "1_1_Darlingtom_open_collector"
+        (path "/05699bf1-a3b3-4463-ad36-cd7a58153539"
+          (reference "R4") (unit 1)
+        )
+      )
+    )
+  )
+  (symbol (lib_id "Device:R") (at 78.74 62.23 90) (unit 1)
+    (in_bom yes) (on_board yes) (dnp no) (fields_autoplaced)
+    (property "Reference" "R3" (at 78.74 55.88 90)
+      (effects (font (size 1.27 1.27)))
+    )
+    (property "Value" "7.2k" (at 78.74 58.42 90)
+      (effects (font (size 1.27 1.27)))
+    )
+    (property "Footprint" "" (at 78.74 64.008 90)
+      (effects (font (size 1.27 1.27)) hide)
+    )
+    (property "Datasheet" "~" (at 78.74 62.23 0)
+      (effects (font (size 1.27 1.27)) hide)
+    )
+    (pin "1")
+    (pin "2")
+    (instances
+      (project "1_1_Darlingtom_open_collector"
+        (path "/05699bf1-a3b3-4463-ad36-cd7a58153539"
+          (reference "R3") (unit 1)
+        )
+      )
