File: Projekti_iz_elektronike/Vsebine/Študijsko_Gradivo/circ/1_1_Komparator.kicad_sch (KiCad schematic)
At the start: 6 parts, among them U1 LM358

Commit message: popravljena vezja
Parts:
- V3: value 5 -> 4.7V
Connections:
- net U_{REF}: now reaches U1.2 (-), V3.1
Other:
- note added: ".tran 1u 6m"
- moved on the sheet: U1A, U1C, V1, V2, V3, V4, V5
