File: Projekti_iz_elektronike/Vsebine/Študijsko_Gradivo/circ/110_Darlingtom_open_collector.kicad_sch (KiCad schematic)
At the start: 10 parts, among them Q1 NPN, Q2 NPN

Commit message: popravljena vezja
Connections:
- net GND: no longer R4.2
- net at Q1.2 (B), Q2.3 (E): no longer R3.2, R4.1
- net at Q2.2 (B), R2.2: no longer R3.1
- new net: R3.2, R4.1
Other:
- note added: "1. Preverite kako hitro lahko TR1 in TR2 prenehata prevajati. 2. Dodajte R3=7.2k in R4=3k k tranzistorjema... (glej ULN2804A) 3. ... in še enkrat preverite napetostne signale."
- note removed: "1. Preverite kako hitro se lahko TR1 in TR2 "zapreta". 2. Dodajte R3=7.2k in R4=3k k tranzistorjema... (glej ULN2804A) 3. ... in še enkrat preverite napetostne signale."
Changed lines of the file:
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@@
 (kicad_sch (version 20230121) (generator eeschema)
-  (paper "A4")
+  (paper "A5")
   (junction (at 97.79 72.39) (diameter 0) (color 0 0 0 0)
   )
@@
   )
   (junction (at 54.61 46.99) (diameter 0) (color 0 0 0 0)
-  )
-  (junction (at 74.93 46.99) (diameter 0) (color 0 0 0 0)
-  )
-  (junction (at 83.82 62.23) (diameter 0) (color 0 0 0 0)
-  )
-  (junction (at 97.79 62.23) (diameter 0) (color 0 0 0 0)
-  )
-  (junction (at 83.82 52.07) (diameter 0) (color 0 0 0 0)
   )
   (wire (pts (xy 38.1 81.28) (xy 38.1 83.82))
@@
     (stroke (width 0) (type default))
   )
-  (wire (pts (xy 74.93 46.99) (xy 74.93 62.23))
-    (stroke (width 0) (type default))
-  )
   (wire (pts (xy 54.61 72.39) (xy 97.79 72.39))
     (stroke (width 0) (type default))
@@
     (stroke (width 0) (type default))
   )
-  (wire (pts (xy 97.79 62.23) (xy 97.79 72.39))
-    (stroke (width 0) (type default))
-  )
-  (wire (pts (xy 74.93 46.99) (xy 76.2 46.99))
+  (wire (pts (xy 71.12 46.99) (xy 76.2 46.99))
     (stroke (width 0) (type default))
   )
@@
     (stroke (width 0) (type default))
   )
-  (wire (pts (xy 83.82 62.23) (xy 86.36 62.23))
-    (stroke (width 0) (type default))
-  )
-  (wire (pts (xy 71.12 46.99) (xy 74.93 46.99))
-    (stroke (width 0) (type default))
-  )
   (wire (pts (xy 110.49 41.91) (xy 110.49 50.8))
     (stroke (width 0) (type default))
@@
     (stroke (width 0) (type default))
   )
-  (wire (pts (xy 83.82 52.07) (xy 83.82 62.23))
-    (stroke (width 0) (type default))
-  )
-  (wire (pts (xy 93.98 62.23) (xy 97.79 62.23))
-    (stroke (width 0) (type default))
-  )
   (wire (pts (xy 54.61 58.42) (xy 54.61 72.39))
     (stroke (width 0) (type default))
@@
     (stroke (width 0) (type default))
   )
-  (wire (pts (xy 97.79 57.15) (xy 97.79 62.23))
+  (wire (pts (xy 97.79 57.15) (xy 97.79 72.39))
     (stroke (width 0) (type default))
   )
-  (wire (pts (xy 82.55 62.23) (xy 83.82 62.23))
+  (wire (pts (xy 82.55 62.23) (xy 86.36 62.23))
     (stroke (width 0) (type default))
   )
@@
     (effects (font (size 1.27 1.27)) (justify left bottom))
   )
-  (text "1. Preverite kako hitro se lahko TR1 in TR2 \"zapreta\".\n2. Dodajte R3=7.2k in R4=3k k tranzistorjema... (glej ULN2804A)\n3. ... in še enkrat preverite napetostne signale."
+  (text "1. Preverite kako hitro lahko TR1 in TR2 prenehata prevajati.\n2. Dodajte R3=7.2k in R4=3k k tranzistorjema... (glej ULN2804A)\n3. ... in še enkrat preverite napetostne signale."
     (at 38.1 34.29 0)
     (effects (font (size 1.27 1.27)) (justify left bottom))

Commit message: thom
Other:
- title: (none) -> Darlington tranzistor-prehod v zaporno stanje
