File: Projekti_iz_elektronike/Vsebine/Študijsko_Gradivo/circ/120_Komparator.kicad_sch (KiCad schematic)
At the start: 6 parts, among them U1 LM741

Commit message: popravljena vezja
Other:
- moved on the sheet: U1, V1, V2, V3, V4, V5
