File: Projekti_iz_elektronike/Vsebine/Študijsko_Gradivo/circ/326_Odstevalnik_LM358_prenos_diferenčnih_signalov.kicad_sch (KiCad schematic)
At the start: 13 parts

Commit message: popravljena vezja
Connections:
- net 0: no longer R1.1
- net GNDREF: now also C2.1, R1.1
- net SIG: now also C1.1
Other:
- moved on the sheet: C1, C2, R1, R2, R3, R4, R5, R8, V1, V2, V4, V5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

Commit message: thom
Parts:
- removed V1: VSIN, symbol Simulation_SPICE:VSIN
- added V3: VTRRANDOM, symbol Simulation_SPICE:VTRRANDOM
Connections:
- net 0: now also V3.2
- net SIG: now also R5.1, V2.1; no longer C1.1, R2.1, R5.2
- net at C1.2, C2.2: now also V3.1
- net GNDREF renamed GND+EM
- net GND+EM: now also C1.1; no longer C2.1
- new net SIG+EM: C2.1, R2.1, R5.2
Other:
- note added: "Daljša razdalja prenosnih signalnih povezav, obremenjena z EM motnjami iz okolice."
- note removed: "Daljša razdalja prenosnih signalnih povezav, obremenjena s EM motnjami iz okolice."
- moved on the sheet: C1, C2, R5, R8
