File: Projekti_iz_elektronike/Vsebine/Študijsko_Gradivo/circ/122_Schmittov_sprožilnik.kicad_sch (KiCad schematic)
At the start: 7 parts, among them U1 LM741

Commit message: popravljena vezja
Other:
- moved on the sheet: R1, R2, U1, V1, V2, V3, V4

Commit message: thom
Parts:
- added V5: 3V, symbol Simulation_SPICE:VDC
Connections:
- net GND: now also V5.2
