File: Projekti_iz_elektronike/Vsebine/Študijsko_Gradivo/circ/311_Vklop_induktivnega_bremena.kicad_sch (KiCad schematic)
At the start: 8 parts, among them Q1 BC108

Commit message: popravljena vezja
Other:
- moved on the sheet: C1, D1, L1, Q1, R1, R2, V1, V2

Commit message: car
Parts:
- C1: value 10uF -> 1 nF
Connections:
- net 0: now also C1.2
- net VTR: now also C1.1
