File: Projekti_iz_elektronike/Vsebine/Študijsko_Gradivo/circ/442_OpAmp_Instrumentacijski_oj_sis_BASIC.kicad_sch (KiCad schematic)
At the start: 17 parts

Commit message: HTOM
Other:
- note added: ".op *.dc V2 0 120 0.5"
- note removed: ".op *.dc V3 0 120 0.5"
