File: Projekti_iz_elektronike/Vsebine/Studijsko_Gradivo/circ/122_Schmittov_sprožilnik.kicad_sch (KiCad schematic)
At the start: 8 parts, among them U1 LM741

Commit message: gradivo
Changed lines of the file:
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@@
 (kicad_sch
-	(version 20231120)
+	(version 20250114)
 	(generator "eeschema")
-	(generator_version "8.0")
+	(generator_version "9.0")
 	(paper "A5")
+	(text ".tran 1m 20m"
+		(exclude_from_sim no)
+		(at 39.37 16.51 0)
+		(effects
+			(font
+				(size 1.27 1.27)
+			)
+			(justify left bottom)
+		)
+	)
 	(junction
 		(at 80.01 27.94)
@@
 		)
 	)
-	(text ".tran 1m 20m"
-		(exclude_from_sim no)
-		(at 39.37 16.51 0)
+	(label "Uin+"
+		(at 57.15 25.4 0)
 		(effects
 			(font
@@
 		)
 	)
-	(label "Uin+"
-		(at 57.15 25.4 0)
-		(fields_autoplaced yes)
-		(effects
-			(font
-				(size 1.27 1.27)
-			)
-			(justify left bottom)
-		)
-	)
 	(label "Uin-"
 		(at 57.15 30.48 0)
-		(fields_autoplaced yes)
 		(effects
 			(font
@@
 		)
 	)
+	(embedded_fonts no)
 )
