File: Projekti_iz_elektronike/Vsebine/Studijsko_Gradivo/circ/326_Odstevalnik_LM358_prenos_diferenčnih_signalov.kicad_sch (KiCad schematic)
At the start: 13 parts

Commit message: rezultati THOM
Changed lines of the file:
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@@
 					(size 1.27 1.27)
 				)
+				(hide yes)
 			)
 		)
@@
 					(size 1.27 1.27)
 				)
-			)
-		)
+				(hide yes)
+			)
+		)
