File: Projekti_iz_elektronike/Vsebine/Studijsko_Gradivo/circ/433_Napake_ojacevalnih_sistemov_Mirovni_Tok.kicad_sch (KiCad schematic)
At the start: 6 parts, among them U1 LM358

Commit message: pripomoček THOM
Parts:
- added R3: 500k, symbol Device:R
Connections:
- net 0: now also R3.2; no longer U1.3 (+)
- new net: R3.1, U1.3 (+)
Changed lines of the file:
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@@
 	(wire
 		(pts
-			(xy 123.19 68.58) (xy 123.19 72.39)
+			(xy 123.19 68.58) (xy 123.19 71.12)
 		)
 		(stroke
@@
 		(pts
 			(xy 24.13 114.3) (xy 27.94 114.3)
+		)
+		(stroke
+			(width 0)
+			(type default)
+		)
+	)
+	(wire
+		(pts
+			(xy 123.19 78.74) (xy 123.19 81.28)
 		)
 		(stroke
@@
 	)
 	(symbol
+		(lib_id "Device:R")
+		(at 123.19 74.93 0)
+		(unit 1)
+		(exclude_from_sim no)
+		(in_bom yes)
+		(on_board yes)
+		(dnp no)
+		(fields_autoplaced yes)
+		(property "Reference" "R3"
+			(at 125.73 73.6599 0)
+			(effects
+				(font
+					(size 1.27 1.27)
+				)
+				(justify left)
+			)
+		)
+		(property "Value" "500k"
+			(at 125.73 76.1999 0)
+			(effects
+				(font
+					(size 1.27 1.27)
+				)
+				(justify left)
+			)
+		)
+		(property "Footprint" ""
+			(at 121.412 74.93 90)
+			(effects
+				(font
+					(size 1.27 1.27)
+				)
+				(hide yes)
+			)
+		)
+		(property "Datasheet" "~"
+			(at 123.19 74.93 0)
+			(effects
+				(font
+					(size 1.27 1.27)
+				)
+				(hide yes)
+			)
+		)
+		(property "Description" ""
+			(at 123.19 74.93 0)
+			(effects
+				(font
+					(size 1.27 1.27)
+				)
+				(hide yes)
+			)
+		)
+		(pin "2"
+		)
+		(pin "1"
+		)
+		(instances
+			(project "433_Napake_ojacevalnih_sistemov_Mirovni_Tok"
+				(path "/f671c449-d824-4cba-8033-5886a9f4776c"
+					(reference "R3")
+					(unit 1)
+				)
+			)
+		)
+	)
+	(symbol
 		(lib_id "Simulation_SPICE:0")
-		(at 123.19 72.39 0)
+		(at 123.19 81.28 0)
 		(unit 1)
 		(exclude_from_sim no)
@@
 		(fields_autoplaced yes)
 		(property "Reference" "#GND01"
-			(at 123.19 74.93 0)
+			(at 123.19 83.82 0)
 			(effects
 				(font
@@
 		)
 		(property "Value" "0"
-			(at 123.19 69.85 0)
+			(at 123.19 78.74 0)
 			(effects
 				(font
@@
 		)
 		(property "Footprint" ""
-			(at 123.19 72.39 0)
+			(at 123.19 81.28 0)
 			(effects
 				(font
@@
 		)
 		(property "Datasheet" "~"
-			(at 123.19 72.39 0)
+			(at 123.19 81.28 0)
 			(effects
 				(font
@@
 		)
 		(property "Description" ""
-			(at 123.19 72.39 0)
-			(effects
-				(font
+			(at 123.19 81.28 0)
+			(effects
+				(font
